File: pcb/eagle/aq_mx_v1-3-0c.brd (EAGLE design)
At the start: 208.6 x 112.5 mm, 37 parts, among them J1 DB9-MALE-RA, J2 DB9-MALE-RA, Q1 BC548, U1 CY62256LL-PC, U2 AY-3-8910, U3 27C512AP, U4 GAL16V8, U5 74LS74N, U6 GAL16V8, U7 74LS244N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

Commit message: Update aq_mx_v1-3-0c.brd
Routing:
- net DE04: track 416.5 -> 417.3 mm
Other:
- outline, holes or cut-outs redrawn
- board text added: "Special thanks to Mack Wharton & Matt Pilz"
- board text added: "v1-3-0, Rev C 01 SEP 2022 by Sean Harrington, sph@1stage.com"
- board text removed: "Aquarius MX v1-3-0 Rev C - 01 SEP 2022 by Sean Harrington, sph@1stage.com"
