File: pcb/eagle/aq_mx_v1-4-0c.sch (EAGLE design)
At the start: 37 parts, among them J1 DB9-MALE-RA, J2 DB9-MALE-RA, Q1 BC548, U1 CY62256LL-PC, U2 AY-3-8910, U3 27C512AP, U4 GAL16V8, U5 74LS74N, U6 GAL16V8, U7 74LS244N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

Commit message: Fix for 1.4.0c PCB
Controller B was missing one of it's mounting holes for metal DB9 ports. If you ordered a PCB with 1.4.0b, you can drill a 1.8" / 3.25mm hole in that position to match the others.
Other:
- note added: "02 FEB 2023"
- note added: "Aquarius MX v1-4-0 - REV C"
- note removed: "21 JAN 2023"
- note removed: "Aquarius MX v1-4-0 - REV B"
Changed lines of the file:
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@@
 <text x="-106.68" y="60.96" size="2.54" layer="97" align="center">Address Buffers</text>
 <text x="-101.6" y="96.52" size="2.54" layer="97" align="center">Balance/Filter Capacitors</text>
-<text x="-101.6" y="-111.76" size="2.286" layer="97" align="center">Aquarius MX v1-4-0 - REV B</text>
+<text x="-101.6" y="-111.76" size="2.286" layer="97" align="center">Aquarius MX v1-4-0 - REV C</text>
 <text x="-101.6" y="-106.68" size="2.54" layer="97" align="center">Project</text>
 <wire x1="-134.62" y1="-114.3" x2="-134.62" y2="-109.22" width="0.1524" layer="97"/>
@@
 <wire x1="-68.58" y1="-114.3" x2="-134.62" y2="-114.3" width="0.1524" layer="97"/>
 <wire x1="-134.62" y1="-109.22" x2="-68.58" y2="-109.22" width="0.1524" layer="97"/>
-<text x="-43.18" y="-111.76" size="2.54" layer="97" align="center">21 JAN 2023</text>
+<text x="-43.18" y="-111.76" size="2.54" layer="97" align="center">02 FEB 2023</text>
 <text x="-43.18" y="-106.68" size="2.54" layer="97" align="center">Revision Date</text>
 <wire x1="-68.58" y1="-114.3" x2="-68.58" y2="-109.22" width="0.1524" layer="97"/>

Commit message: Housekeeping Updates
Other:
- note added: "15 MAR 2023"
- note removed: "02 FEB 2023"
Changed lines of the file:
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@@
 <wire x1="-68.58" y1="-114.3" x2="-134.62" y2="-114.3" width="0.1524" layer="97"/>
 <wire x1="-134.62" y1="-109.22" x2="-68.58" y2="-109.22" width="0.1524" layer="97"/>
-<text x="-43.18" y="-111.76" size="2.54" layer="97" align="center">02 FEB 2023</text>
+<text x="-43.18" y="-111.76" size="2.54" layer="97" align="center">15 MAR 2023</text>
 <text x="-43.18" y="-106.68" size="2.54" layer="97" align="center">Revision Date</text>
 <wire x1="-68.58" y1="-114.3" x2="-68.58" y2="-109.22" width="0.1524" layer="97"/>

Commit message: Minor PCB Tweaks
Other:
- note added: "25 MAR 2023"
- note removed: "15 MAR 2023"
Changed lines of the file:
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@@
 <wire x1="-68.58" y1="-114.3" x2="-134.62" y2="-114.3" width="0.1524" layer="97"/>
 <wire x1="-134.62" y1="-109.22" x2="-68.58" y2="-109.22" width="0.1524" layer="97"/>
-<text x="-43.18" y="-111.76" size="2.54" layer="97" align="center">15 MAR 2023</text>
+<text x="-43.18" y="-111.76" size="2.54" layer="97" align="center">25 MAR 2023</text>
 <text x="-43.18" y="-106.68" size="2.54" layer="97" align="center">Revision Date</text>
 <wire x1="-68.58" y1="-114.3" x2="-68.58" y2="-109.22" width="0.1524" layer="97"/>
